File: PID.kicad_sch (KiCad schematic)
At the start: 29 parts, among them U1 TL072, U2 TL072, U3 TL072, U4 TL072

Commit message: KiCAD sch 60
Parts:
- removed R53: 10k, Resistor_SMD:R_0603_1608Metric_Pad0.98x0.95mm_HandSolder, symbol Device:R
- added C9: 330p, Resistor_SMD:R_0603_1608Metric_Pad0.98x0.95mm_HandSolder, symbol Device:C
- added R27, R28: 22k, Resistor_SMD:R_0603_1608Metric_Pad0.98x0.95mm_HandSolder, symbol Device:R
- added R54: 10k, Resistor_SMD:R_0603_1608Metric_Pad0.98x0.95mm_HandSolder, symbol Device:R
Connections:
- net at U1.7, U4.6 (-): now also C9.1, R54.1
- net at U1.1: now also R27.2, R28.1; no longer U1.6 (-)
- net at U1.3 (+): now also R27.1, R54.2
- new net: C9.2, R28.2, U1.6 (-)
Other:
- note added: "output = (-2.6, 2.6)"
- moved on the sheet: C36, C37, U1A, U1B, U1C
