File: PID_demo.kicad_sch (KiCad schematic)
At the start: 7 parts

Commit message: sim update
Parts:
- added U1: TL072, Package_SO:SOIC-8_3.9x4.9mm_P1.27mm, symbol Amplifier_Operational:TL072
Other:
- moved on the sheet: RV4, RV5

Commit message: KiCAD start
Parts:
- removed H1, H2: MountingHole, PID_lib:M3_hole_with_spacer, symbol Mechanical:MountingHole
- removed RV1, RV2, RV3, RV4, RV5: R_Potentiometer, PID_lib:front_plate_pot, symbol Device:R_Potentiometer
- removed U1: TL072, Package_SO:SOIC-8_3.9x4.9mm_P1.27mm, symbol Amplifier_Operational:TL072
Other:
- added sheet Charge pump (./power_supply.kicad_sch)
- added sheet Motor drive (motor_drive.kicad_sch)
- added sheet PID (PID.kicad_sch)
- title: (none) -> Petnički EKG

Commit message: KiCAD sch 60
Changed lines of the file:
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@@
 	(wire
 		(pts
-			(xy 171.45 44.45) (xy 170.18 44.45)
+			(xy 78.74 62.23) (xy 77.47 62.23)
 		)
 		(stroke
@@
 	(wire
 		(pts
-			(xy 152.4 54.61) (xy 154.94 54.61)
+			(xy 59.69 72.39) (xy 62.23 72.39)
 		)
 		(stroke
@@
 	(wire
 		(pts
-			(xy 153.67 44.45) (xy 154.94 44.45)
+			(xy 60.96 62.23) (xy 62.23 62.23)
 		)
 		(stroke
@@
 	(symbol
 		(lib_id "power:VCC")
-		(at 153.67 44.45 90)
+		(at 60.96 62.23 90)
 		(unit 1)
 		(body_style 1)
@@
 		(fields_autoplaced yes)
 		(property "Reference" "#PWR09"
-			(at 157.48 44.45 0)
+			(at 64.77 62.23 0)
 			(hide yes)
 			(show_name no)
@@
 		)
 		(property "Value" "+5V"
-			(at 149.86 44.4501 90)
+			(at 57.15 62.2301 90)
 			(show_name no)
 			(do_not_autoplace no)
@@
 		)
 		(property "Footprint" ""
-			(at 153.67 44.45 0)
+			(at 60.96 62.23 0)
 			(hide yes)
 			(show_name no)
@@
 		)
 		(property "Datasheet" ""
-			(at 153.67 44.45 0)
+			(at 60.96 62.23 0)
 			(hide yes)
 			(show_name no)
@@
 		)
 		(property "Description" "Power symbol creates a global label with name \"VCC\""
-			(at 153.67 44.45 0)
+			(at 60.96 62.23 0)
 			(hide yes)
 			(show_name no)
@@
 	(symbol
 		(lib_id "Simulation_SPICE:0")
-		(at 152.4 54.61 270)
+		(at 59.69 72.39 270)
 		(unit 1)
 		(body_style 1)
@@
 		(fields_autoplaced yes)
 		(property "Reference" "#GND01"
-			(at 149.86 54.61 0)
+			(at 57.15 72.39 0)
 			(hide yes)
 			(show_name no)
@@
 		)
 		(property "Value" "0"
-			(at 154.94 54.61 0)
+			(at 62.23 72.39 0)
 			(hide yes)
 			(show_name no)
@@
 		)
 		(property "Footprint" ""
-			(at 152.4 54.61 0)
+			(at 59.69 72.39 0)
 			(hide yes)
 			(show_name no)
@@
 		)
 		(property "Datasheet" ""
-			(at 152.4 54.61 0)
+			(at 59.69 72.39 0)
 			(hide yes)
 			(show_name no)
@@
 		)
 		(property "Description" ""
-			(at 152.4 54.61 0)
+			(at 59.69 72.39 0)
 			(hide yes)
 			(show_name no)
@@
 	(symbol
 		(lib_id "power:VCC")
-		(at 171.45 44.45 270)
+		(at 78.74 62.23 270)
 		(unit 1)
 		(body_style 1)
@@
 		(dnp no)
 		(property "Reference" "#PWR010"
-			(at 167.64 44.45 0)
+			(at 74.93 62.23 0)
 			(hide yes)
 			(show_name no)
@@
 		)
 		(property "Value" "-5V"
-			(at 175.26 44.45 90)
+			(at 82.55 62.23 90)
 			(show_name no)
 			(do_not_autoplace no)
@@
 		)
 		(property "Footprint" ""
-			(at 171.45 44.45 0)
+			(at 78.74 62.23 0)
 			(hide yes)
 			(show_name no)
@@
 		)
 		(property "Datasheet" ""
-			(at 171.45 44.45 0)
+			(at 78.74 62.23 0)
 			(hide yes)
 			(show_name no)
@@
 		)
 		(property "Description" "Power symbol creates a global label with name \"VCC\""
-			(at 171.45 44.45 0)
+			(at 78.74 62.23 0)
 			(hide yes)
 			(show_name no)
@@
 	)
 	(sheet
-		(at 154.94 41.91)
+		(at 62.23 59.69)
 		(size 15.24 15.24)
 		(exclude_from_sim no)
@@
 		)
 		(property "Sheetname" "Charge pump"
-			(at 154.94 41.1984 0)
+			(at 62.23 58.9784 0)
 			(show_name no)
 			(do_not_autoplace no)
@@
 		)
 		(property "Sheetfile" "./power_supply.kicad_sch"
-			(at 154.94 57.7346 0)
+			(at 62.23 75.5146 0)
 			(show_name no)
 			(do_not_autoplace no)
@@
 		)
 		(pin "GND" input
-			(at 154.94 54.61 180)
+			(at 62.23 72.39 180)
 			(effects
 				(font
@@
 		)
 		(pin "-5V" output
-			(at 170.18 44.45 0)
+			(at 77.47 62.23 0)
 			(effects
 				(font
@@
 		)
 		(pin "+5V" input
-			(at 154.94 44.45 180)
-			(effects
-				(font
+			(at 62.23 62.23 180)
+			(effects
+				(font
