File: motor_drive.kicad_sch (KiCad schematic)
At the start: 23 parts, among them Q11 AO3401A, Q15 AO3400A, Q16 AO3400A, Q9 AO3401A, U8 74HC14

Commit message: KiCAD sch 60
Other:
- note added: "PWM generation"
- note removed: "CLK generation"
- moved on the sheet: Q11, Q16, Q9
