File: PID_demo.kicad_pcb (KiCad board)
At the start: 2 copper layers, 100 x 100 mm, 7 parts

Commit message: KiCAD start
Parts:
- removed H1, H2: MountingHole, PID_lib:M3_hole_with_spacer
- added C1: 10u, Resistor_SMD:R_0805_2012Metric_Pad1.20x1.40mm_HandSolder, B.Cu at (134.5, 62.4)
- added C10: 10u, Resistor_SMD:R_0805_2012Metric_Pad1.20x1.40mm_HandSolder, B.Cu at (149.0, 63.0)
- added C11: 10u, Resistor_SMD:R_0805_2012Metric_Pad1.20x1.40mm_HandSolder, F.Cu at (80.4, 133.9)
- added C17: 1n, Capacitor_SMD:C_0603_1608Metric_Pad1.08x0.95mm_HandSolder, B.Cu at (157.7, 71.8)
- added C2: 10u, Resistor_SMD:R_0805_2012Metric_Pad1.20x1.40mm_HandSolder, B.Cu at (141.8, 59.4)
- added C31: 100n, Capacitor_SMD:C_0603_1608Metric_Pad1.08x0.95mm_HandSolder, B.Cu at (148.8, 61.3)
- added C32: 100n, Capacitor_SMD:C_0603_1608Metric_Pad1.08x0.95mm_HandSolder, F.Cu at (71.0, 138.7)
- added C35: 100n, Capacitor_SMD:C_0603_1608Metric_Pad1.08x0.95mm_HandSolder, B.Cu at (134.7, 67.9)
- added C4: 100n, Capacitor_SMD:C_0603_1608Metric_Pad1.08x0.95mm_HandSolder, B.Cu at (138.2, 58.3)
- added C41: 10u, Resistor_SMD:R_0805_2012Metric_Pad1.20x1.40mm_HandSolder, B.Cu at (141.8, 70.4)
- added C42: 100n, Capacitor_SMD:C_0603_1608Metric_Pad1.08x0.95mm_HandSolder, B.Cu at (138.2, 71.4)
- added C43: 10u, Resistor_SMD:R_0805_2012Metric_Pad1.20x1.40mm_HandSolder, B.Cu at (141.8, 68.5)
- added C44: 10u, Resistor_SMD:R_0805_2012Metric_Pad1.20x1.40mm_HandSolder, F.Cu at (21.7, 106.6)
- added C46: 1u, Capacitor_SMD:C_0603_1608Metric_Pad1.08x0.95mm_HandSolder, B.Cu at (151.7, 66.7)
- added C47: 1u, Capacitor_SMD:C_0603_1608Metric_Pad1.08x0.95mm_HandSolder, F.Cu at (71.0, 141.2)
- added C49: 10u, Resistor_SMD:R_0805_2012Metric_Pad1.20x1.40mm_HandSolder, B.Cu at (141.8, 61.3)
- added C5: 100p, Capacitor_SMD:C_0603_1608Metric_Pad1.08x0.95mm_HandSolder, B.Cu at (153.3, 69.2)
- added C50: 10u, Resistor_SMD:R_0805_2012Metric_Pad1.20x1.40mm_HandSolder, B.Cu at (141.8, 63.2)
- added C51: 10u, Resistor_SMD:R_0805_2012Metric_Pad1.20x1.40mm_HandSolder, B.Cu at (134.5, 58.6)
- added C52: 10u, Resistor_SMD:R_0805_2012Metric_Pad1.20x1.40mm_HandSolder, B.Cu at (134.5, 60.5)
- added C53: 10u, Resistor_SMD:R_0805_2012Metric_Pad1.20x1.40mm_HandSolder, B.Cu at (134.5, 64.3)
- added C54: 10u, Resistor_SMD:R_0805_2012Metric_Pad1.20x1.40mm_HandSolder, B.Cu at (134.5, 66.2)
- added C55: 10u, Resistor_SMD:R_0805_2012Metric_Pad1.20x1.40mm_HandSolder, B.Cu at (149.0, 64.9)
- added C56: 10u, Resistor_SMD:R_0805_2012Metric_Pad1.20x1.40mm_HandSolder, B.Cu at (149.0, 66.8)
- added C57: 10u, Resistor_SMD:R_0805_2012Metric_Pad1.20x1.40mm_HandSolder, B.Cu at (149.0, 68.7)
- added C58: 10u, Resistor_SMD:R_0805_2012Metric_Pad1.20x1.40mm_HandSolder, B.Cu at (149.0, 70.6)
- added C59: 10u, Resistor_SMD:R_0805_2012Metric_Pad1.20x1.40mm_HandSolder, F.Cu at (80.4, 136.8)
- added C6: 100p, Capacitor_SMD:C_0603_1608Metric_Pad1.08x0.95mm_HandSolder, F.Cu at (71.0, 133.7)
- added C60: 100n, Capacitor_SMD:C_0603_1608Metric_Pad1.08x0.95mm_HandSolder, B.Cu at (141.8, 64.9)
- added C61: 10u, Resistor_SMD:R_0805_2012Metric_Pad1.20x1.40mm_HandSolder, F.Cu at (80.4, 139.8)
- added C62: 10u, Resistor_SMD:R_0805_2012Metric_Pad1.20x1.40mm_HandSolder, F.Cu at (80.4, 142.7)
- added C63: 10u, Resistor_SMD:R_0805_2012Metric_Pad1.20x1.40mm_HandSolder, F.Cu at (80.4, 145.7)
- added C65: 10u, Resistor_SMD:R_0805_2012Metric_Pad1.20x1.40mm_HandSolder, B.Cu at (141.8, 66.6)
- added C7: 100p, Capacitor_SMD:C_0603_1608Metric_Pad1.08x0.95mm_HandSolder, B.Cu at (151.7, 63.3)
- added C8: 100p, Capacitor_SMD:C_0603_1608Metric_Pad1.08x0.95mm_HandSolder, F.Cu at (71.0, 136.2)
- added D10: 1N4148WS, Diode_SMD:D_SOD-323, B.Cu at (159.4, 71.8)
- added D11: 1N4148WS, Diode_SMD:D_SOD-323, B.Cu at (163.4, 65.7)
- added D12: 1N4148WS, Diode_SMD:D_SOD-323, B.Cu at (163.4, 63.7)
- added D13: 1N4148WS, Diode_SMD:D_SOD-323, B.Cu at (138.2, 69.7)
- added D14: 1N4148WS, Diode_SMD:D_SOD-323, F.Cu at (89.6, 133.9)
- added D15: 1N4148WS, Diode_SMD:D_SOD-323, F.Cu at (89.6, 136.8)
- added D16: 1N4148WS, Diode_SMD:D_SOD-323, F.Cu at (89.6, 139.8)
- added D3: GREEN_LED, LED_SMD:LED_0805_2012Metric_Pad1.15x1.40mm_HandSolder, B.Cu at (152.4, 58.8)
- added D4: GREEN_LED, LED_SMD:LED_0805_2012Metric_Pad1.15x1.40mm_HandSolder, F.Cu at (75.6, 151.7)
- added D8: 1N4148WS, Diode_SMD:D_SOD-323, B.Cu at (138.2, 60.0)
- added D9: 1N4148WS, Diode_SMD:D_SOD-323, B.Cu at (163.6, 72.8)
- added J1: Conn_01x04_Pin, Connector_PinHeader_2.54mm:PinHeader_1x04_P2.54mm_Vertical, F.Cu at (143.1, 74.1)
- added JP5: Jumper_2_Open, Jumper:SolderJumper-2_P1.3mm_Open_RoundedPad1.0x1.5mm, B.Cu at (163.5, 70.1)
- added Q10: AO3401A, Package_TO_SOT_SMD:SOT-23, B.Cu at (138.2, 62.9)
- added Q11: AO3401A, Package_TO_SOT_SMD:SOT-23, F.Cu at (75.6, 139.1)
- added Q13: AO3400A, Package_TO_SOT_SMD:SOT-23, B.Cu at (145.4, 66.9)
- added Q14: AO3400A, Package_TO_SOT_SMD:SOT-23, B.Cu at (138.2, 66.8)
- added Q15: AO3400A, Package_TO_SOT_SMD:SOT-23, F.Cu at (75.6, 143.5)
- added Q16: AO3400A, Package_TO_SOT_SMD:SOT-23, F.Cu at (75.6, 148.0)
- added Q8: AO3401A, Package_TO_SOT_SMD:SOT-23, B.Cu at (145.4, 63.0)
- added Q9: AO3401A, Package_TO_SOT_SMD:SOT-23, F.Cu at (75.6, 134.6)
- added R1: 1k, Resistor_SMD:R_0603_1608Metric_Pad0.98x0.95mm_HandSolder, B.Cu at (148.8, 59.0)
- added R10: 1k, Resistor_SMD:R_0603_1608Metric_Pad0.98x0.95mm_HandSolder, F.Cu at (71.0, 146.2)
- added R11: 1k, Resistor_SMD:R_0603_1608Metric_Pad0.98x0.95mm_HandSolder, F.Cu at (71.0, 148.7)
- added R2: 1k, Resistor_SMD:R_0603_1608Metric_Pad0.98x0.95mm_HandSolder, F.Cu at (71.0, 143.7)
- added R37: 100k, Resistor_SMD:R_0603_1608Metric_Pad0.98x0.95mm_HandSolder, B.Cu at (161.2, 71.8)
- added R38: 100k, Resistor_SMD:R_0603_1608Metric_Pad0.98x0.95mm_HandSolder, B.Cu at (163.6, 74.6)
- added R40: 10k, Resistor_SMD:R_0603_1608Metric_Pad0.98x0.95mm_HandSolder, B.Cu at (163.4, 67.4)
- added R41: 10k, Resistor_SMD:R_0603_1608Metric_Pad0.98x0.95mm_HandSolder, F.Cu at (71.0, 151.2)
- added R42: 10k, Resistor_SMD:R_0603_1608Metric_Pad0.98x0.95mm_HandSolder, F.Cu at (71.0, 153.7)
- added R43: 10k, Resistor_SMD:R_0603_1608Metric_Pad0.98x0.95mm_HandSolder, F.Cu at (17.1, 106.4)
- added R44: 10k, Resistor_SMD:R_0603_1608Metric_Pad0.98x0.95mm_HandSolder, F.Cu at (17.1, 108.9)
- added R45: 10k, Resistor_SMD:R_0603_1608Metric_Pad0.98x0.95mm_HandSolder, F.Cu at (17.1, 111.4)
- added R46: 10k, Resistor_SMD:R_0603_1608Metric_Pad0.98x0.95mm_HandSolder, F.Cu at (17.1, 113.9)
- added R47: 10k, Resistor_SMD:R_0603_1608Metric_Pad0.98x0.95mm_HandSolder, F.Cu at (17.1, 116.4)
- added R48: 10k, Resistor_SMD:R_0603_1608Metric_Pad0.98x0.95mm_HandSolder, F.Cu at (17.1, 118.9)
- added R49: 10k, Resistor_SMD:R_0603_1608Metric_Pad0.98x0.95mm_HandSolder, F.Cu at (17.1, 121.4)
- added R50: 10k, Resistor_SMD:R_0603_1608Metric_Pad0.98x0.95mm_HandSolder, F.Cu at (17.1, 123.9)
- added R51: 20k, Resistor_SMD:R_0603_1608Metric_Pad0.98x0.95mm_HandSolder, B.Cu at (160.5, 69.2)
- added R9: 1k, Resistor_SMD:R_0603_1608Metric_Pad0.98x0.95mm_HandSolder, B.Cu at (163.4, 62.0)
- added U1: TL072, Package_SO:SOIC-8_3.9x4.9mm_P1.27mm, F.Cu at (10.7, 108.5)
- added U2: TL072, Package_SO:SOIC-8_3.9x4.9mm_P1.27mm, F.Cu at (10.7, 115.0)
- added U3: TL072, Package_SO:SOIC-8_3.9x4.9mm_P1.27mm, F.Cu at (10.7, 121.6)
- added U4: TL072, Package_SO:SOIC-8_3.9x4.9mm_P1.27mm, F.Cu at (10.7, 128.2)
- added U7: 74HC14, Package_SO:SOIC-14_3.9x8.7mm_P1.27mm, B.Cu at (157.1, 64.7)
- added U8: 74HC14, Package_SO:SOIC-14_3.9x8.7mm_P1.27mm, F.Cu at (87.0, 149.9)
- moved RV1 50.2 mm to (115.0, 100.0)
- moved RV2 50.2 mm to (150.0, 100.0)
- moved RV3 50.2 mm to (185.0, 100.0)
- moved RV4 50.2 mm to (115.0, 65.0)
- moved RV5 50.2 mm to (185.0, 66.0)
Routing:
- net PMOS_GATE: track 0.00 -> 32.2 mm
- net NMOS_GATE: track 0.00 -> 30.5 mm
- net 0: track 0.00 -> 22.6 mm, vias 0 -> 17
- net Net-(D12-A): track 0.00 -> 19.2 mm
- net +5V: track 0.00 -> 17.8 mm, vias 0 -> 2
- net /Charge pump/MID_DRV: track 0.00 -> 17.2 mm
- net /Charge pump/MID_REC: track 0.00 -> 16.5 mm
- net Net-(D11-K): track 0.00 -> 15.1 mm
- net CLK: track 0.00 -> 12.0 mm
- net -5V: track 0.00 -> 11.0 mm, vias 0 -> 1
- net Net-(D10-A): track 0.00 -> 6.90 mm
- net Net-(D13-A): track 0.00 -> 4.25 mm
- net Net-(D9-A): track 0.00 -> 4.24 mm
- net Net-(D10-K): track 0.00 -> 3.93 mm
- net Net-(D8-A): track 0.00 -> 3.75 mm
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- added copper zone on B.Cu, net 0
- added copper zone on F.Cu, net 0
Other:
- board text added: "BAT-"

Commit message: KiCAD sch 60
Parts:
- added C33: 100n, Capacitor_SMD:C_0603_1608Metric_Pad1.08x0.95mm_HandSolder, F.Cu at (1.68, 3.27)
- added C34: 100n, Capacitor_SMD:C_0603_1608Metric_Pad1.08x0.95mm_HandSolder, F.Cu at (1.68, 5.78)
- added C36: 100n, Capacitor_SMD:C_0603_1608Metric_Pad1.08x0.95mm_HandSolder, F.Cu at (1.68, 8.29)
- added C37: 100n, Capacitor_SMD:C_0603_1608Metric_Pad1.08x0.95mm_HandSolder, F.Cu at (1.68, 10.8)
- added C38: 100n, Capacitor_SMD:C_0603_1608Metric_Pad1.08x0.95mm_HandSolder, F.Cu at (6.03, 0.76)
- added C39: 100n, Capacitor_SMD:C_0603_1608Metric_Pad1.08x0.95mm_HandSolder, F.Cu at (6.03, 3.27)
- added C40: 100n, Capacitor_SMD:C_0603_1608Metric_Pad1.08x0.95mm_HandSolder, F.Cu at (6.03, 5.78)
- added C45: 10u, Resistor_SMD:R_0805_2012Metric_Pad1.20x1.40mm_HandSolder, F.Cu at (1.88, 13.5)
- added C48: 100n, Capacitor_SMD:C_0603_1608Metric_Pad1.08x0.95mm_HandSolder, F.Cu at (6.03, 8.29)
- added C9: 330p, Resistor_SMD:R_0603_1608Metric_Pad0.98x0.95mm_HandSolder, F.Cu at (1.68, 0.76)
- added R27: 22k, Resistor_SMD:R_0603_1608Metric_Pad0.98x0.95mm_HandSolder, F.Cu at (6.03, 10.8)
- added R28: 22k, Resistor_SMD:R_0603_1608Metric_Pad0.98x0.95mm_HandSolder, F.Cu at (10.4, 0.76)
- added R52: 10k, Resistor_SMD:R_0603_1608Metric_Pad0.98x0.95mm_HandSolder, F.Cu at (10.4, 3.27)
- added R54: 10k, Resistor_SMD:R_0603_1608Metric_Pad0.98x0.95mm_HandSolder, F.Cu at (10.4, 5.78)
- RV4: value R_Potentiometer -> position
- RV5: value R_Potentiometer -> target
- moved C41 70.8 mm to (111.8, 134.5)
- moved C43 70.8 mm to (111.8, 132.6)
- moved C55 70.8 mm to (119.0, 129.0)
- moved C60 70.8 mm to (111.8, 129.0)
- moved Q13 70.8 mm to (115.4, 131.0)
- moved R40 70.8 mm to (133.4, 131.5)
- moved C1 70.8 mm to (104.5, 126.5)
- moved C10 70.8 mm to (119.0, 127.1)
- moved C2 70.8 mm to (111.8, 123.5)
- moved C31 70.8 mm to (118.8, 125.4)
- moved C35 70.8 mm to (104.7, 132.0)
- moved C4 70.8 mm to (108.2, 122.4)
- moved C42 70.8 mm to (108.2, 135.5)
- moved C46 70.8 mm to (121.7, 130.7)
- moved C49 70.8 mm to (111.8, 125.4)
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Connections:
- C44 pad 1: unconnected-(C44-Pad1) -> Net-(U3A--)
- C44 pad 2: unconnected-(C44-Pad2) -> Net-(C44-Pad2)
- R44 pad 2: Net-(R44-Pad2) -> Net-(C44-Pad2)
- R47 pad 2: unconnected-(R47-Pad2) -> Net-(R47-Pad2)
- R48 pad 1: Net-(U3A--) -> Net-(C45-Pad1)
- R49 pad 2: unconnected-(R49-Pad2) -> Net-(R49-Pad2)
- RV1 pad 1: unconnected-(RV1-Pad1) -> Net-(R45-Pad2)
- RV1 pad 2: unconnected-(RV1-Pad2) -> Net-(U2B--)
- RV1 pad 3: unconnected-(RV1-Pad3) -> Net-(U2B--)
- RV2 pad 1: unconnected-(RV2-Pad1) -> Net-(C45-Pad1)
- RV2 pad 2: unconnected-(RV2-Pad2) -> Net-(U3A--)
- RV2 pad 3: unconnected-(RV2-Pad3) -> Net-(U3A--)
- RV3 pad 1: unconnected-(RV3-Pad1) -> Net-(U3B--)
- RV3 pad 2: unconnected-(RV3-Pad2) -> Net-(R43-Pad2)
- RV3 pad 3: unconnected-(RV3-Pad3) -> Net-(R43-Pad2)
- RV4 pad 1: unconnected-(RV4-Pad1) -> +5V
- RV4 pad 2: unconnected-(RV4-Pad2) -> Net-(R47-Pad2)
- RV4 pad 3: unconnected-(RV4-Pad3) -> -5V
- RV5 pad 1: unconnected-(RV5-Pad1) -> +5V
- RV5 pad 2: unconnected-(RV5-Pad2) -> Net-(R49-Pad2)
- RV5 pad 3: unconnected-(RV5-Pad3) -> -5V
- U1 pad 1: Net-(U1B--) -> Net-(R27-Pad2)
- U1 pad 3: unconnected-(U1A-+-Pad3) -> Net-(U1A-+)
- U1 pad 4: unconnected-(U1C-V--Pad4) -> -5V
- U1 pad 8: unconnected-(U1C-V+-Pad8) -> +5V
- U2 pad 1: Net-(U3A--) -> Net-(C45-Pad1)
- U2 pad 4: unconnected-(U2C-V--Pad4) -> -5V
- U2 pad 6: unconnected-(U2B---Pad6) -> Net-(U2B--)
- U2 pad 8: unconnected-(U2C-V+-Pad8) -> +5V
- U3 pad 1: Net-(R44-Pad2) -> Net-(C44-Pad2)
- U3 pad 4: unconnected-(U3C-V--Pad4) -> -5V
- U3 pad 6: unconnected-(U3B---Pad6) -> Net-(U3B--)
- U3 pad 8: unconnected-(U3C-V+-Pad8) -> +5V
- U4 pad 4: unconnected-(U4C-V--Pad4) -> -5V
- U4 pad 7: /PID/PWM -> /Motor drive/PWM
- U4 pad 8: unconnected-(U4C-V+-Pad8) -> +5V
Other:
- board text added: "MOTOR"

Commit message: KiCAD sch - motor added
Parts:
- added M1: Motor_DC, PID_lib:N20_motor, F.Cu at (150.0, 65.0)
Changed lines of the file:
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@@
+		)
+	)
+	(footprint "PID_lib:N20_motor"
+		(layer "F.Cu")
+		(at 150 65)
+		(descr "Potentiometer, vertical, bottom-adjust, single slot, Bourns 3314R-1, http://www.bourns.com/docs/Product-Datasheets/3314.pdf")
+		(tags "Potentiometer vertical hole Bourns 3314R-1")
+		(property "Reference" "M1"
+			(at 0 -4.65 0)
+			(layer "B.SilkS")
+			(hide yes)
+			(effects
+				(font
+					(size 1 1)
+					(thickness 0.15)
+				)
+			)
+		)
+		(property "Value" "Motor_DC"
+			(at 0 4.65 0)
+			(layer "F.Fab")
+			(effects
+				(font
+					(size 1 1)
+					(thickness 0.15)
+				)
+			)
+		)
+		(property "Datasheet" ""
+			(at 0 0 0)
+			(unlocked yes)
+			(layer "F.Fab")
+			(hide yes)
+			(effects
+				(font
+					(size 1.27 1.27)
+					(thickness 0.15)
+				)
+			)
+		)
+		(property "Description" "DC Motor"
+			(at 0 0 0)
+			(unlocked yes)
+			(layer "F.Fab")
+			(hide yes)
+			(effects
+				(font
+					(size 1.27 1.27)
+					(thickness 0.15)
+				)
+			)
+		)
+		(property ki_fp_filters "PinHeader*P2.54mm* TerminalBlock*")
+		(sheetname "/Charge pump/")
+		(sheetfile "./power_supply.kicad_sch")
+		(units
+			(unit
+				(name "A")
+				(pins "1" "2")
+			)
+		)
+		(attr smd)
+		(duplicate_pad_numbers_are_jumpers no)
+		(fp_line
+			(start -0.24 -2.37)
+			(end 0.24 -2.37)
+			(stroke
+				(width 0.12)
+				(type solid)
+			)
+			(layer "F.SilkS")
+		)
+		(fp_rect
+			(start -6 -5)
+			(end 6 5)
+			(stroke
+				(width 0.1)
+				(type default)
+			)
+			(fill no)
+			(layer "B.SilkS")
+		)
+		(fp_rect
+			(start -6.75 -5.5)
+			(end 6.75 5.5)
+			(stroke
+				(width 0.05)
+				(type default)
+			)
+			(fill no)
+			(layer "B.CrtYd")
+		)
+		(fp_rect
+			(start -5.75 -2.75)
+			(end 5.75 2.75)
+			(stroke
+				(width 0.05)
+				(type default)
+			)
+			(fill no)
+			(layer "F.CrtYd")
+		)
+		(fp_line
+			(start -2.5 -2.25)
+			(end -2.5 2.25)
+			(stroke
+				(width 0.1)
+				(type solid)
+			)
+			(layer "F.Fab")
+		)
+		(fp_line
+			(start -2.5 2.25)
+			(end 2.5 2.25)
+			(stroke
+				(width 0.1)
+				(type solid)
+			)
+			(layer "F.Fab")
+		)
+		(fp_line
+			(start 2.5 -2.25)
+			(end -2.5 -2.25)
+			(stroke
+				(width 0.1)
+				(type solid)
+			)
+			(layer "F.Fab")
+		)
+		(fp_line
+			(start 2.5 2.25)
+			(end 2.5 -2.25)
+			(stroke
+				(width 0.1)
+				(type solid)
+			)
+			(layer "F.Fab")
+		)
+		(fp_text user "${REFERENCE}"
+			(at 0 -1.7 0)
+			(layer "F.Fab")
+			(effects
+				(font
+					(size 0.63 0.63)
+					(thickness 0.15)
+				)
+			)
+		)
+		(pad "MH" thru_hole circle
+			(at -4.4 0)
+			(size 2 2)
+			(drill 2)
+			(layers "*.Cu" "*.Mask")
+			(remove_unused_layers no)
+		)
+		(pad "MH" thru_hole circle
+			(at 0 0)
+			(size 5 5)
+			(drill 5)
+			(layers "*.Cu" "*.Mask")
+			(remove_unused_layers no)
+		)
+		(pad "MH" thru_hole circle
+			(at 4.4 0)
+			(size 2 2)
+			(drill 2)
+			(layers "*.Cu" "*.Mask")
+			(remove_unused_layers no)
+		)
+		(embedded_fonts no)
+		(model "${KIPRJMOD}/PID_lib.pretty/N20 Mini Micro Metall Gear Motor.step"
+			(offset
+				(xyz 0 0 -11.5)
+			)
+			(scale
+				(xyz 1 1 1)
+			)
+			(rotate
+				(xyz -90 90 -0)
+			)
 		)
 	)

Commit message: KiCAD sch - note
Other:
- board text added: "naglasiti P I D komponente i na silkscreen-u na poledjini"
Changed lines of the file:
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@@
 		(layer "Edge.Cuts")
+	)
+	(gr_text "naglasiti P I D komponente i na silkscreen-u na poledjini"
+		(at 188 122 0)
+		(layer "B.Cu")
+		(effects
+			(font
+				(size 1.5 1.5)
+				(thickness 0.3)
+				(bold yes)
+			)
+			(justify left bottom mirror)
+		)
 	)
 	(gr_text "BAT-"
